File: Latch_Rasp.kicad_pcb (KiCad board)
At the start: 2 copper layers, 22.1 x 20.3 mm, 19 parts, among them J2 Conn_02x03_Counter_Clockwise, J5 USB_C_Receptacle_PowerOnly_6P, Q1 NDT456P, Q2 AO3414, SW1 SW_Push

Commit message: wip
Parts:
- added C2: 10n, Capacitor_SMD:C_0805_2012Metric, B.Cu at (124.0, 81.3)
- R1: value 100K -> 5.1K
Routing:
- net /Q2G: track 21.9 -> 23.6 mm
Changed lines of the file:
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@@
 			)
 		)
-		(property "Value" "100K"
+		(property "Value" "5.1K"
 			(at 0 1.65 0)
 			(layer "F.Fab")
@@
 		)
 		(property "Sim.Device" "NMOS"
-			(at 0 0 -90)
+			(at 0 0 270)
 			(unlocked yes)
 			(layer "F.Fab")
@@
 		)
 		(property "Sim.Type" "VDMOS"
-			(at 0 0 -90)
+			(at 0 0 270)
 			(unlocked yes)
 			(layer "F.Fab")
@@
 		)
 		(property "Sim.Pins" "1=D 2=G 3=S"
-			(at 0 0 -90)
+			(at 0 0 270)
 			(unlocked yes)
 			(layer "F.Fab")
@@
 		(sheetname "/")
 		(sheetfile "Latch_Rasp.kicad_sch")
-		(attr through_hole)
 		(fp_line
 			(start -1.38 -1.38)
@@
 		)
 	)
+	(footprint "Capacitor_SMD:C_0805_2012Metric"
+		(layer "B.Cu")
+		(at 123.952 81.28 180)
+		(descr "Capacitor SMD 0805 (2012 Metric), square (rectangular) end terminal, IPC-7351 nominal, (Body size source: IPC-SM-782 page 76, https://www.pcb-3d.com/wordpress/wp-content/uploads/ipc-sm-782a_amendment_1_and_2.pdf, https://docs.google.com/spreadsheets/d/1BsfQQcO9C6DZCsRaXUlFlo91Tg2WpOkGARC1WS5S8t0/edit?usp=sharing), generated with kicad-footprint-generator")
+		(tags "capacitor")
+		(property "Reference" "C2"
+			(at 0 1.68 0)
+			(layer "B.SilkS")
+			(effects
+				(font
+					(size 1 1)
+					(thickness 0.15)
+				)
+				(justify mirror)
+			)
+		)
+		(property "Value" "10n"
+			(at 0 -1.68 0)
+			(layer "B.Fab")
+			(effects
+				(font
+					(size 1 1)
+					(thickness 0.15)
+				)
+				(justify mirror)
+			)
+		)
+		(property "Datasheet" "~"
+			(at 0 0 0)
+			(layer "B.Fab")
+			(hide yes)
+			(effects
+				(font
+					(size 1.27 1.27)
+					(thickness 0.15)
+				)
+				(justify mirror)
+			)
+		)
+		(property "Description" "Unpolarized capacitor"
+			(at 0 0 0)
+			(layer "B.Fab")
+			(hide yes)
+			(effects
+				(font
+					(size 1.27 1.27)
+					(thickness 0.15)
+				)
+				(justify mirror)
+			)
+		)
+		(property ki_fp_filters "C_*")
+		(sheetname "/")
+		(sheetfile "Latch_Rasp.kicad_sch")
+		(attr smd)
+		(fp_line
+			(start -0.261252 0.735)
+			(end 0.261252 0.735)
+			(stroke
+				(width 0.12)
+				(type solid)
+			)
+			(layer "B.SilkS")
+		)
+		(fp_line
+			(start -0.261252 -0.735)
+			(end 0.261252 -0.735)
+			(stroke
+				(width 0.12)
+				(type solid)
+			)
+			(layer "B.SilkS")
+		)
+		(fp_line
+			(start 1.7 0.98)
+			(end 1.7 -0.98)
+			(stroke
+				(width 0.05)
+				(type solid)
+			)
+			(layer "B.CrtYd")
+		)
+		(fp_line
+			(start 1.7 -0.98)
+			(end -1.7 -0.98)
+			(stroke
+				(width 0.05)
+				(type solid)
+			)
+			(layer "B.CrtYd")
+		)
+		(fp_line
+			(start -1.7 0.98)
+			(end 1.7 0.98)
+			(stroke
+				(width 0.05)
+				(type solid)
+			)
+			(layer "B.CrtYd")
+		)
+		(fp_line
+			(start -1.7 -0.98)
+			(end -1.7 0.98)
+			(stroke
+				(width 0.05)
+				(type solid)
+			)
+			(layer "B.CrtYd")
+		)
+		(fp_line
+			(start 1 0.625)
+			(end 1 -0.625)
+			(stroke
+				(width 0.1)
+				(type solid)
+			)
+			(layer "B.Fab")
+		)
+		(fp_line
+			(start 1 -0.625)
+			(end -1 -0.625)
+			(stroke
+				(width 0.1)
+				(type solid)
+			)
+			(layer "B.Fab")
+		)
+		(fp_line
+			(start -1 0.625)
+			(end 1 0.625)
+			(stroke
+				(width 0.1)
+				(type solid)
+			)
+			(layer "B.Fab")
+		)
+		(fp_line
+			(start -1 -0.625)
+			(end -1 0.625)
+			(stroke
+				(width 0.1)
+				(type solid)
+			)
+			(layer "B.Fab")
+		)
+		(fp_text user "${REFERENCE}"
+			(at 0 0 0)
+			(layer "B.Fab")
+			(effects
+				(font
+					(size 0.5 0.5)
+					(thickness 0.08)
+				)
+				(justify mirror)
+			)
+		)
+		(pad "1" smd roundrect
+			(at -0.95 0 180)
+			(size 1 1.45)
+			(layers "B.Cu" "B.Mask" "B.Paste")
+			(roundrect_rratio 0.25)
+			(net 9 "/Q2G")
+			(pintype "passive")
+		)
+		(pad "2" smd roundrect
+			(at 0.95 0 180)
+			(size 1 1.45)
+			(layers "B.Cu" "B.Mask" "B.Paste")
+			(roundrect_rratio 0.25)
+			(net 3 "GND")
+			(pintype "passive")
+		)
+		(embedded_fonts no)
+		(model "${KICAD9_3DMODEL_DIR}/Capacitor_SMD.3dshapes/C_0805_2012Metric.step"
+			(offset
+				(xyz 0 0 0)
+			)
+			(scale
+				(xyz 1 1 1)
+			)
+			(rotate
+				(xyz 0 0 0)
+			)
+		)
+	)
 	(footprint "Connector_PinSocket_2.54mm:PinSocket_2x05_P2.54mm_Vertical"
 		(layer "B.Cu")
@@
 		(tags "resistor")
 		(property "Reference" "R4"
-			(at 0.795628 1.61181 0)
+			(at 2.954628 0.508 0)
 			(layer "B.SilkS")
 			(effects
@@
 	)
 	(segment
-		(start 124.771128 82.861128)
-		(end 122.682 80.772)
+		(start 124.648 81.28)
+		(end 123.124 79.756)
 		(width 0.3)
 		(layer "B.Cu")
@@
 	)
 	(segment
-		(start 124.771128 83.566)
-		(end 124.771128 82.861128)
+		(start 120.396 79.756)
+		(end 119.38 80.772)
 		(width 0.3)
 		(layer "B.Cu")
@@
 	)
 	(segment
-		(start 126.528128 83.566)
-		(end 124.771128 83.566)
+		(start 124.771128 81.403128)
+		(end 124.648 81.28)
 		(width 0.3)
 		(layer "B.Cu")
@@
 	)
 	(segment
-		(start 122.682 80.772)
-		(end 119.38 80.772)
+		(start 123.124 79.756)
+		(end 120.396 79.756)
+		(width 0.3)
+		(layer "B.Cu")
+		(net 9)
+	)
+	(segment
+		(start 124.771128 83.566)
+		(end 124.771128 81.403128)
+		(width 0.3)
+		(layer "B.Cu")
+		(net 9)
+	)
+	(segment
+		(start 126.528128 83.566)
+		(end 124.771128 83.566)
 		(width 0.3)
 		(layer "B.Cu")
